File: Eagle CadSoft Design files/GB SOP32 ROM Adapter mini version.sch (EAGLE design)
At the start: 7 parts, among them IC1 AM29F016/32

Commit message: first commit
Parts:
- removed !R, !WE: TPTP08SQ, testpad:TPTP08SQ
- added WE: TPTP06SQ, testpad:TPTP06SQ
- A20, A21: value TPTP08SQ -> TPTP06SQ; device testpad:TPTP08SQ -> testpad:TPTP06SQ
- IC1: device jrodrigo-gameboy:AM29FXXXTSOP48-STANDARD -> jrodrigo-gameboy:AM29FXXXTSOP48_WITHOUT_NC
Connections:
- removed net !RESET: !R.TP, IC1.!RESET
- net !WE: now also WE.TP; no longer !WE.TP
- net VCC: now also IC1.!RESET
